File: KITE_CTRL.kicad_sch (KiCad schematic)
At the start: 0 parts

Commit message: Selected battery charger
Parts:
- added J?: PICO, PICO, symbol PICO:PICO
- added U?: MCP73812T-420I-OT, Package_TO_SOT_SMD:SOT-23-5, symbol Battery_Management:MCP73812T-420I-OT
Changed lines of the file:
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@@
 (kicad_sch (version 20210621) (generator eeschema)
   (paper "A4")
-  (symbol_instances)
+  (symbol (lib_id "Battery_Management:MCP73812T-420I-OT") (at 210.82 57.15 0) (unit 1)
+    (in_bom yes) (on_board yes) (fields_autoplaced)
+    (property "Reference" "U?" (id 0) (at 221.6151 56.2415 0)
+      (effects (font (size 1.27 1.27)) (justify left))
+    )
+    (property "Value" "MCP73812T-420I-OT" (id 1) (at 221.6151 59.0166 0)
+      (effects (font (size 1.27 1.27)) (justify left))
+    )
+    (property "Footprint" "Package_TO_SOT_SMD:SOT-23-5" (id 2) (at 212.09 63.5 0)
+      (effects (font (size 1.27 1.27)) (justify left) hide)
+    )
+    (property "Datasheet" "http://ww1.microchip.com/downloads/en/DeviceDoc/22036b.pdf" (id 3) (at 204.47 50.8 0)
+      (effects (font (size 1.27 1.27)) hide)
+    )
+    (pin "1")
+    (pin "2")
+    (pin "3")
+    (pin "4")
+    (pin "5")
+  )
+  (symbol (lib_id "PICO:PICO") (at 129.54 95.25 0) (unit 1)
+    (in_bom yes) (on_board yes) (fields_autoplaced)
+    (property "Reference" "J?" (id 0) (at 147.32 163.3126 0))
+    (property "Value" "PICO" (id 1) (at 147.32 166.0877 0))
+    (property "Footprint" "PICO" (id 2) (at 161.29 39.37 0)
+      (effects (font (size 1.27 1.27)) (justify left) hide)
+    )
+    (property "Datasheet" "https://datasheets.raspberrypi.org/pico/pico_datasheet.pdf" (id 3) (at 161.29 41.91 0)
+      (effects (font (size 1.27 1.27)) (justify left) hide)
+    )
+    (property "Description" "RP2040 microcontroller chip designed by Raspberry Pi in the United Kingdom 2  SPI, 2  I2C, 2  UART, 3  12-bit ADC, 16  controllable PWM channels" (id 4) (at 161.29 44.45 0)
+      (effects (font (size 1.27 1.27)) (justify left) hide)
+    )
+    (property "Height" "1" (id 5) (at 161.29 46.99 0)
+      (effects (font (size 1.27 1.27)) (justify left) hide)
+    )
+    (property "Manufacturer_Name" "RASPBERRY-PI" (id 6) (at 161.29 49.53 0)
+      (effects (font (size 1.27 1.27)) (justify left) hide)
+    )
+    (property "Manufacturer_Part_Number" "PICO" (id 7) (at 161.29 52.07 0)
+      (effects (font (size 1.27 1.27)) (justify left) hide)
+    )
+    (property "Mouser Part Number" "" (id 8) (at 161.29 54.61 0)
+      (effects (font (size 1.27 1.27)) (justify left) hide)
+    )
+    (property "Mouser Price/Stock" "" (id 9) (at 161.29 57.15 0)
+      (effects (font (size 1.27 1.27)) (justify left) hide)
+    )
+    (property "Arrow Part Number" "" (id 10) (at 161.29 59.69 0)
+      (effects (font (size 1.27 1.27)) (justify left) hide)
+    )
+    (property "Arrow Price/Stock" "" (id 11) (at 161.29 62.23 0)
+      (effects (font (size 1.27 1.27)) (justify left) hide)
+    )
+    (pin "1")
+    (pin "10")
+    (pin "11")
+    (pin "12")
+    (pin "13")
+    (pin "14")
+    (pin "15")
+    (pin "16")
+    (pin "17")
+    (pin "18")
+    (pin "19")
+    (pin "2")
+    (pin "20")
+    (pin "21")
+    (pin "22")
+    (pin "23")
+    (pin "24")
+    (pin "25")
+    (pin "26")
+    (pin "27")
+    (pin "28")
+    (pin "29")
+    (pin "3")
+    (pin "30")
+    (pin "31")
+    (pin "32")
+    (pin "33")
+    (pin "34")
+    (pin "35")
+    (pin "36")
+    (pin "37")
+    (pin "38")
+    (pin "39")
+    (pin "4")
+    (pin "40")
+    (pin "5")
+    (pin "6")
+    (pin "7")
+    (pin "8")
+    (pin "9")
+    (pin "D1")
+    (pin "D2")
+    (pin "D3")
+    (pin "TP1")
+    (pin "TP2")
+    (pin "TP3")
+    (pin "TP4")
+    (pin "TP5")
+    (pin "TP6")
+  )
+  (sheet_instances
+    (path "/" (page "1"))
+  )
+  (symbol_instances
+    (path "/cc22a68a-31e5-4e7e-ad19-8e64ee28b102"
+      (reference "J?") (unit 1) (value "PICO") (footprint "PICO")
+    )
+    (path "/cdc473e3-7a52-440a-a3a5-0e5c3e6d8005"
+      (reference "U?") (unit 1) (value "MCP73812T-420I-OT") (footprint "Package_TO_SOT_SMD:SOT-23-5")
+    )
+  )
 )
