File: KITE_CTRL.kicad_pcb (KiCad board)
At the start: 0 parts

Commit message: Finnished laying out the board
Parts:
- added C1: 1uF, Capacitor_SMD:C_0402_1005Metric, B.Cu at (145.0, 67.0)
- added C2: 1uF, Capacitor_SMD:C_0402_1005Metric, B.Cu at (136.0, 77.1)
- added D2: D_Schottky, Diode_SMD:D_0402_1005Metric, B.Cu at (146.6, 69.4)
- added J1: PICO, KiCad:PICO, F.Cu at (128.9, 116.8)
- added J2: LED_STRIP, Connector_PinSocket_2.54mm:PinSocket_1x03_P2.54mm_Vertical, F.Cu at (134.6, 74.4)
- added J3: BATTERY, S2B-PH-SM4-TB_LF__SN_:JST_S2B-PH-SM4-TB(LF)(SN), B.Cu at (141.1, 78.6)
- added R1: 2kR, Resistor_SMD:R_0402_1005Metric, B.Cu at (144.0, 73.7)
- added SW1: MASTER, PCM12SMTR:SW_PCM12SMTR, B.Cu at (137.0, 68.0)
- added U1: MCP73812T-420I-OT, Package_TO_SOT_SMD:SOT-23-5, B.Cu at (144.0, 71.0)
Routing:
- net -BATT: track 0.00 -> 73.6 mm, vias 0 -> 5
- net +BATT: track 0.00 -> 29.3 mm, vias 0 -> 2
- net NEO_PIN: track 0.00 -> 15.3 mm
- net Net-(J1-Pad37): track 0.00 -> 14.4 mm, vias 0 -> 1
- net +5V: track 0.00 -> 13.1 mm, vias 0 -> 3
- net Net-(J1-Pad39): track 0.00 -> 4.09 mm, vias 0 -> 1
- net Net-(R1-Pad1): track 0.00 -> 1.81 mm
Other:
- board outline added: 24.6 x 22.1 mm
- copper layers 0 -> 2
